Commit message: Updates.

File: rpn/create_dataset/models/new/brown_bowl/models/textured.urdf (robot description, URDF)
Before this commit: robot textured, 1 links, 0 joints
Links:
- link base_link: geometry collision mesh filename=model_normalized.obj scale=0.35 0.35 0.35; visual mesh filename=model_normalized.obj scale=0.35 0.35 0.35

File: rpn/create_dataset/models/new/coke_bottle/models/textured.urdf (robot description, URDF)
Before this commit: robot textured, 1 links, 0 joints
Links:
- link base_link: geometry collision mesh filename=model_normalized.obj scale=0.3 0.3 0.3; visual mesh filename=model_normalized.obj scale=0.3 0.3 0.3

File: rpn/create_dataset/models/new/powerade/models/textured.urdf (robot description, URDF)
Before this commit: robot textured, 1 links, 0 joints
Links:
- link base_link: geometry collision mesh filename=model_normalized.obj scale=0.32 0.32 0.32; visual mesh filename=model_normalized.obj scale=0.32 0.32 0.32

File: rpn/create_dataset/models/new/wine_bottle/models/textured.urdf (robot description, URDF)
Before this commit: robot textured, 1 links, 0 joints
Links:
- link base_link: geometry collision mesh filename=model_normalized.obj scale=0.3 0.3 0.3; visual mesh filename=model_normalized.obj scale=0.3 0.3 0.3
